File: _autosave-telemetry-pcb.sch (KiCad schematic (older format))
At the start: 44 parts, among them CN1 12V_IN, CN10 THERMO1, CN11 THERMO2, CN12 RS232, CN13 CAN, CN14 CAN, CN15 12V_OUT, CN16 12V_OUT, CN2 12V_OUT, CN3 12V_OUT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

Commit message: laid out all components and got most footprints imported
Parts:
- CN10, CN11: footprint (none) -> Conn_Molex_70553-0002:Molex-70553-0002-0-0-0; symbol Connector_Generic:Conn_01x02 -> Connector_Generic:Conn_01x03
- CN13, CN14, CN6, CN7, CN8, CN9: footprint (none) -> Conn_Molex_70553-0001:Molex-70553-0001-0-0-MFG
Connections:
- no-connect marks 16 -> 18
Changed lines of the file:
@@
 F 0 "CN6" V 7314 112 50  0000 R CNN
 F 1 "CAN" V 7223 112 50  0000 R CNN
-F 2 "" H 7350 300 50  0001 C CNN
+F 2 "Conn_Molex_70553-0001:Molex-70553-0001-0-0-MFG" H 7350 300 50  0001 C CNN
 F 3 "~" H 7350 300 50  0001 C CNN
 	1    7350 300
@@
 F 0 "CN7" V 8114 112 50  0000 R CNN
 F 1 "CAN" V 8023 112 50  0000 R CNN
-F 2 "" H 8150 300 50  0001 C CNN
+F 2 "Conn_Molex_70553-0001:Molex-70553-0001-0-0-MFG" H 8150 300 50  0001 C CNN
 F 3 "~" H 8150 300 50  0001 C CNN
 	1    8150 300
@@
 F 0 "CN8" V 8864 112 50  0000 R CNN
 F 1 "CAN" V 8773 112 50  0000 R CNN
-F 2 "" H 8900 300 50  0001 C CNN
+F 2 "Conn_Molex_70553-0001:Molex-70553-0001-0-0-MFG" H 8900 300 50  0001 C CNN
 F 3 "~" H 8900 300 50  0001 C CNN
 	1    8900 300
@@
 F 0 "CN9" V 9614 112 50  0000 R CNN
 F 1 "CAN" V 9523 112 50  0000 R CNN
-F 2 "" H 9650 300 50  0001 C CNN
+F 2 "Conn_Molex_70553-0001:Molex-70553-0001-0-0-MFG" H 9650 300 50  0001 C CNN
 F 3 "~" H 9650 300 50  0001 C CNN
 	1    9650 300
@@
 F 0 "CN13" V 10314 112 50  0000 R CNN
 F 1 "CAN" V 10223 112 50  0000 R CNN
-F 2 "" H 10350 300 50  0001 C CNN
+F 2 "Conn_Molex_70553-0001:Molex-70553-0001-0-0-MFG" H 10350 300 50  0001 C CNN
 F 3 "~" H 10350 300 50  0001 C CNN
 	1    10350 300
@@
 F 0 "CN14" V 10964 112 50  0000 R CNN
 F 1 "CAN" V 10873 112 50  0000 R CNN
-F 2 "" H 11000 300 50  0001 C CNN
+F 2 "Conn_Molex_70553-0001:Molex-70553-0001-0-0-MFG" H 11000 300 50  0001 C CNN
 F 3 "~" H 11000 300 50  0001 C CNN
 	1    11000 300
@@
 Wire Wire Line
 	3050 6000 2500 6000
-Wire Wire Line
-	2500 6000 2500 5800
 Connection ~ 3050 6000
 $Comp
@@
 Wire Wire Line
 	3050 4900 2500 4900
-Wire Wire Line
-	2500 4900 2500 4700
 Connection ~ 3050 4900
 Wire Wire Line
@@
 $EndComp
 $Comp
-L Connector_Generic:Conn_01x02 CN10
+L Connector_Generic:Conn_01x03 CN11
+U 1 1 601BC25C
+P 2300 5800
+F 0 "CN11" V 2264 5612 50  0000 R CNN
+F 1 "THERMO2" V 2173 5612 50  0000 R CNN
+F 2 "Conn_Molex_70553-0002:Molex-70553-0002-0-0-0" H 2300 5800 50  0001 C CNN
+F 3 "~" H 2300 5800 50  0001 C CNN
+	1    2300 5800
+	-1   0    0    1
+$EndComp
+Connection ~ 1400 700
+Wire Wire Line
+	1400 1000 1400 1200
+Wire Wire Line
+	1200 1350 1200 500
+Wire Wire Line
+	1200 1350 1100 1350
+Connection ~ 1200 1350
+Wire Wire Line
+	1100 500  1100 600
+Wire Wire Line
+	1600 1350 2250 1350
+Wire Wire Line
+	750  1350 1100 1350
+Connection ~ 1100 1350
+Wire Wire Line
+	750  1250 750  1200
+Wire Wire Line
+	750  1200 1400 1200
+Connection ~ 1400 1200
+Wire Wire Line
+	2250 1350 3100 1350
+Connection ~ 1400 600
+Wire Wire Line
+	1400 600  1400 700
+Wire Wire Line
+	2150 1200 3000 1200
+Connection ~ 1100 600
+Wire Wire Line
+	1100 600  1100 1350
+Wire Wire Line
+	1400 1200 1850 1200
+Wire Wire Line
+	1850 1100 1850 1200
+Connection ~ 1850 1200
+Wire Wire Line
+	1850 1200 2150 1200
+Wire Wire Line
+	2500 4800 2500 4900
+Wire Wire Line
+	2500 5900 2500 6000
+NoConn ~ 2500 4700
+NoConn ~ 2500 5800
+$Comp
+L Connector_Generic:Conn_01x03 CN10
 U 1 1 60178289
 P 2300 4700
 F 0 "CN10" V 2264 4512 50  0000 R CNN
 F 1 "THERMO1" V 2173 4512 50  0000 R CNN
-F 2 "" H 2300 4700 50  0001 C CNN
+F 2 "Conn_Molex_70553-0002:Molex-70553-0002-0-0-0" H 2300 4700 50  0001 C CNN
 F 3 "~" H 2300 4700 50  0001 C CNN
 	1    2300 4700
 	-1   0    0    1
 $EndComp
-$Comp
-L Connector_Generic:Conn_01x02 CN11
-U 1 1 601BC25C
-P 2300 5800
-F 0 "CN11" V 2264 5612 50  0000 R CNN
-F 1 "THERMO2" V 2173 5612 50  0000 R CNN
-F 2 "" H 2300 5800 50  0001 C CNN
-F 3 "~" H 2300 5800 50  0001 C CNN
-	1    2300 5800
-	-1   0    0    1
-$EndComp
-Connection ~ 1400 700
-Wire Wire Line
-	1400 1000 1400 1200
-Wire Wire Line
-	1200 1350 1200 500
-Wire Wire Line
-	1200 1350 1100 1350
-Connection ~ 1200 1350
-Wire Wire Line
-	1100 500  1100 600
-Wire Wire Line
-	1600 1350 2250 1350
-Wire Wire Line
-	750  1350 1100 1350
-Connection ~ 1100 1350
-Wire Wire Line
-	750  1250 750  1200
-Wire Wire Line
-	750  1200 1400 1200
-Connection ~ 1400 1200
-Wire Wire Line
-	2250 1350 3100 1350
-Connection ~ 1400 600
-Wire Wire Line
-	1400 600  1400 700
-Wire Wire Line
-	2150 1200 3000 1200
-Connection ~ 1100 600
-Wire Wire Line
-	1100 600  1100 1350
-Wire Wire Line
-	1400 1200 1850 1200
-Wire Wire Line
-	1850 1100 1850 1200
-Connection ~ 1850 1200
-Wire Wire Line
-	1850 1200 2150 1200
 $EndSCHEMATC
