File: spi.sch (KiCad schematic (older format))
At the start: 19 parts, among them CN14 THERMO1, CN15 THERMO2, IC2 MAX31855K, IC3 MAX31855K, IC4 MCP2515-xSO, IC5 TCAN332DR, IC6 LSM6DSOTR, Y1 8MHz

Commit message: finished schematic and PCB layout for 1.1 board
Parts:
- added CN7, CN8: CAN, telemetry-pcb:molex_sl_1x02_horizontal, symbol Connector_Generic:Conn_01x02
- added R9: 120, Resistor_SMD:R_0805_2012Metric, symbol Device:R
- added S2: CAN_TERM, Button_Switch_THT:SW_DIP_SPSTx01_Piano_10.8x4.1mm_W7.62mm_P2.54mm, symbol Switch:SW_DIP_x01
- added T6: TEST_CAN, TestPoint:TestPoint_2Pads_Pitch2.54mm_Drill0.8mm, symbol Connector:Conn_01x02_Female
- renumbered CN14 to CN5, CN15 to CN6
Connections:
- net labels removed: CANH, CANL
- wire segments 127 -> 141
Changed lines of the file:
@@
 $Descr A4 11693 8268
 encoding utf-8
-Sheet 4 4
+Sheet 3 3
 Title ""
 Date ""
@@
 P 4550 7800
 AR Path="/6196EF4B" Ref="#PWR?"  Part="1"
-AR Path="/6195E29D/6196EF4B" Ref="#PWR0121"  Part="1"
-F 0 "#PWR0121" H 4550 7550 50  0001 C CNN
+AR Path="/6195E29D/6196EF4B" Ref="#PWR021"  Part="1"
+F 0 "#PWR021" H 4550 7550 50  0001 C CNN
 F 1 "GND" H 4555 7627 50  0000 C CNN
 F 2 "" H 4550 7800 50  0001 C CNN
@@
 P 8600 7300
 AR Path="/6196EF73" Ref="#PWR?"  Part="1"
-AR Path="/6195E29D/6196EF73" Ref="#PWR0122"  Part="1"
-F 0 "#PWR0122" H 8600 7050 50  0001 C CNN
+AR Path="/6195E29D/6196EF73" Ref="#PWR025"  Part="1"
+F 0 "#PWR025" H 8600 7050 50  0001 C CNN
 F 1 "GND" H 8605 7127 50  0000 C CNN
 F 2 "" H 8600 7300 50  0001 C CNN
@@
 P 8600 5950
 AR Path="/6197F71A" Ref="#PWR?"  Part="1"
-AR Path="/6195E29D/6197F71A" Ref="#PWR0123"  Part="1"
-F 0 "#PWR0123" H 8600 5800 50  0001 C CNN
+AR Path="/6195E29D/6197F71A" Ref="#PWR024"  Part="1"
+F 0 "#PWR024" H 8600 5800 50  0001 C CNN
 F 1 "+3V3" H 8615 6123 50  0000 C CNN
 F 2 "" H 8600 5950 50  0001 C CNN
@@
 P 4550 5700
 AR Path="/6197F723" Ref="#PWR?"  Part="1"
-AR Path="/6195E29D/6197F723" Ref="#PWR0124"  Part="1"
-F 0 "#PWR0124" H 4550 5550 50  0001 C CNN
+AR Path="/6195E29D/6197F723" Ref="#PWR020"  Part="1"
+F 0 "#PWR020" H 4550 5550 50  0001 C CNN
 F 1 "+3V3" H 4565 5873 50  0000 C CNN
 F 2 "" H 4550 5700 50  0001 C CNN
@@
 P 1500 950
 AR Path="/6198C074" Ref="#PWR?"  Part="1"
-AR Path="/6195E29D/6198C074" Ref="#PWR0125"  Part="1"
-F 0 "#PWR0125" H 1500 800 50  0001 C CNN
+AR Path="/6195E29D/6198C074" Ref="#PWR016"  Part="1"
+F 0 "#PWR016" H 1500 800 50  0001 C CNN
 F 1 "+3V3" H 1515 1123 50  0000 C CNN
 F 2 "" H 1500 950 50  0001 C CNN
@@
 P 450 1750
 AR Path="/6198C0AA" Ref="CN?"  Part="1"
-AR Path="/6195E29D/6198C0AA" Ref="CN14"  Part="1"
-F 0 "CN14" V 414 1562 50  0000 R CNN
+AR Path="/6195E29D/6198C0AA" Ref="CN5"  Part="1"
+F 0 "CN5" V 414 1562 50  0000 R CNN
 F 1 "THERMO1" V 323 1562 50  0000 R CNN
 F 2 "telemetry-pcb:molex-sl-1x03-horizontal" H 450 1750 50  0001 C CNN
@@
 Wire Wire Line
 	2750 7650 4550 7650
-Text HLabel 10400 5300 2    100  Output ~ 0
-CANH
-Text HLabel 10400 5050 2    100  Output ~ 0
-CANL
 Text HLabel 1600 5950 0    100  Output ~ 0
 MO1
@@
 CAN_INT
 Wire Wire Line
-	6700 6350 6700 5300
-Wire Wire Line
-	6700 5300 10400 5300
-Wire Wire Line
-	6550 6550 6550 5050
-Wire Wire Line
-	6550 5050 10400 5050
+	6700 6350 6700 5500
 Wire Wire Line
 	6550 6550 6850 6550
@@
 P 1500 2100
 AR Path="/61D1474E" Ref="#PWR?"  Part="1"
-AR Path="/6195E29D/61D1474E" Ref="#PWR0126"  Part="1"
-F 0 "#PWR0126" H 1500 1850 50  0001 C CNN
+AR Path="/6195E29D/61D1474E" Ref="#PWR017"  Part="1"
+F 0 "#PWR017" H 1500 1850 50  0001 C CNN
 F 1 "GND" H 1505 1927 50  0000 C CNN
 F 2 "" H 1500 2100 50  0001 C CNN
@@
 	1000 1650 1900 1650
 $Comp
-L telemetry-pcb-rescue:LSM6DSOTR-2021-11-02_20-37-28-telemetry-pcb-rescue-telemetry-pcb-rescue IC6
+L telemetry-pcb-rescue:LSM6DSOTR-2021-11-02_20-37-28-telemetry-pcb-rescue-telemetry-pcb-rescue IC?
 U 1 1 61D40F93
 P 8450 2750
-AR Path="/61D40F93" Ref="IC6"  Part="1"
+AR Path="/61D40F93" Ref="IC?"  Part="1"
 AR Path="/6195E29D/61D40F93" Ref="IC6"  Part="1"
 F 0 "IC6" H 9450 3137 60  0000 C CNN
@@
 P 7250 2450
 AR Path="/61D4578D" Ref="#PWR?"  Part="1"
-AR Path="/6195E29D/61D4578D" Ref="#PWR0127"  Part="1"
-F 0 "#PWR0127" H 7250 2300 50  0001 C CNN
+AR Path="/6195E29D/61D4578D" Ref="#PWR022"  Part="1"
+F 0 "#PWR022" H 7250 2300 50  0001 C CNN
 F 1 "+3V3" H 7265 2623 50  0000 C CNN
 F 2 "" H 7250 2450 50  0001 C CNN
@@
 P 7900 3900
 AR Path="/61D49663" Ref="#PWR?"  Part="1"
-AR Path="/6195E29D/61D49663" Ref="#PWR0128"  Part="1"
-F 0 "#PWR0128" H 7900 3650 50  0001 C CNN
+AR Path="/6195E29D/61D49663" Ref="#PWR023"  Part="1"
+F 0 "#PWR023" H 7900 3650 50  0001 C CNN
 F 1 "GND" H 7905 3727 50  0000 C CNN
 F 2 "" H 7900 3900 50  0001 C CNN
@@
 Text HLabel 4350 650  1    100  Output ~ 0
 SCK
-Text HLabel 7250 750  1    100  Output ~ 0
+Text HLabel 10900 750  1    100  Output ~ 0
 MO
 Text HLabel 4800 650  1    100  Output ~ 0
 MI
-Text HLabel 7650 750  1    100  Output ~ 0
+Text HLabel 11300 750  1    100  Output ~ 0
 IMU_CS
 Text HLabel 5250 650  1    100  Output ~ 0
@@
 P 2200 2900
 AR Path="/61D0AFB5" Ref="#PWR?"  Part="1"
-AR Path="/6195E29D/61D0AFB5" Ref="#PWR0129"  Part="1"
-F 0 "#PWR0129" H 2200 2750 50  0001 C CNN
+AR Path="/6195E29D/61D0AFB5" Ref="#PWR018"  Part="1"
+F 0 "#PWR018" H 2200 2750 50  0001 C CNN
 F 1 "+3V3" H 2215 3073 50  0000 C CNN
 F 2 "" H 2200 2900 50  0001 C CNN
@@
 P 1100 3750
 AR Path="/6198C0A0" Ref="CN?"  Part="1"
-AR Path="/6195E29D/6198C0A0" Ref="CN15"  Part="1"
-F 0 "CN15" V 1064 3562 50  0000 R CNN
+AR Path="/6195E29D/6198C0A0" Ref="CN6"  Part="1"
+F 0 "CN6" V 1064 3562 50  0000 R CNN
 F 1 "THERMO2" V 973 3562 50  0000 R CNN
 F 2 "telemetry-pcb:molex-sl-1x03-horizontal" H 1100 3750 50  0001 C CNN
@@
 P 2200 4150
 AR Path="/6198C06E" Ref="#PWR?"  Part="1"
-AR Path="/6195E29D/6198C06E" Ref="#PWR0130"  Part="1"
-F 0 "#PWR0130" H 2200 3900 50  0001 C CNN
+AR Path="/6195E29D/6198C06E" Ref="#PWR019"  Part="1"
+F 0 "#PWR019" H 2200 3900 50  0001 C CNN
 F 1 "GND" H 2205 3977 50  0000 C CNN
 F 2 "" H 2200 4150 50  0001 C CNN
@@
 Connection ~ 4800 1650
 Wire Wire Line
-	10450 2750 10450 1350
-Wire Wire Line
-	10450 1350 7250 1350
-Wire Wire Line
-	7250 1350 7250 750
-Wire Wire Line
-	7650 750  11300 750
-Wire Wire Line
 	11300 750  11300 2950
 Wire Wire Line
 	11300 2950 10450 2950
+$Comp
+L Connector:Conn_01x02_Female T?
+U 1 1 62470705
+P 10000 5100
+AR Path="/62470705" Ref="T?"  Part="1"
+AR Path="/6188C66E/62470705" Ref="T?"  Part="1"
+AR Path="/6195E29D/62470705" Ref="T6"  Part="1"
+F 0 "T6" H 10028 5076 50  0000 L CNN
+F 1 "TEST_CAN" H 10028 4985 50  0000 L CNN
+F 2 "TestPoint:TestPoint_2Pads_Pitch2.54mm_Drill0.8mm" H 10000 5100 50  0001 C CNN
+F 3 "~" H 10000 5100 50  0001 C CNN
+	1    10000 5100
+	1    0    0    -1
+$EndComp
+$Comp
+L Connector_Generic:Conn_01x02 CN?
+U 1 1 6247070B
+P 10950 4800
+AR Path="/6247070B" Ref="CN?"  Part="1"
+AR Path="/6188C66E/6247070B" Ref="CN?"  Part="1"
+AR Path="/6195E29D/6247070B" Ref="CN7"  Part="1"
+F 0 "CN7" V 10914 4612 50  0000 R CNN
+F 1 "CAN" V 10823 4612 50  0000 R CNN
+F 2 "telemetry-pcb:molex_sl_1x02_horizontal" H 10950 4800 50  0001 C CNN
+F 3 "~" H 10950 4800 50  0001 C CNN
+	1    10950 4800
+	1    0    0    -1
+$EndComp
+$Comp
+L Switch:SW_DIP_x01 S?
+U 1 1 62470711
+P 8350 5250
+AR Path="/62470711" Ref="S?"  Part="1"
+AR Path="/6188C66E/62470711" Ref="S?"  Part="1"
+AR Path="/6195E29D/62470711" Ref="S2"  Part="1"
+F 0 "S2" H 8350 5517 50  0000 C CNN
+F 1 "CAN_TERM" H 8350 5426 50  0000 C CNN
+F 2 "Button_Switch_THT:SW_DIP_SPSTx01_Piano_10.8x4.1mm_W7.62mm_P2.54mm" H 8350 5250 50  0001 C CNN
+F 3 "~" H 8350 5250 50  0001 C CNN
+	1    8350 5250
+	1    0    0    -1
+$EndComp
+$Comp
+L Device:R R?
+U 1 1 62470717
+P 8950 5050
+AR Path="/62470717" Ref="R?"  Part="1"
+AR Path="/6188C66E/62470717" Ref="R?"  Part="1"
+AR Path="/6195E29D/62470717" Ref="R9"  Part="1"
+F 0 "R9" V 9157 5050 50  0000 C CNN
+F 1 "120" V 9066 5050 50  0000 C CNN
+F 2 "Resistor_SMD:R_0805_2012Metric" V 8880 5050 50  0001 C CNN
+F 3 "~" H 8950 5050 50  0001 C CNN
+	1    8950 5050
+	-1   0    0    1
+$EndComp
+Wire Wire Line
+	10450 2750 10900 2750
+Wire Wire Line
+	10900 2750 10900 750
+Wire Wire Line
+	6550 4800 6550 6550
+Wire Wire Line
+	9800 5200 9800 5500
+Wire Wire Line
+	9800 5100 9800 4800
+Connection ~ 9800 4800
+Connection ~ 9800 5500
+Wire Wire Line
+	6700 5500 8050 5500
+Wire Wire Line
+	6550 4800 8950 4800
+Wire Wire Line
+	9800 5500 10450 5500
+Wire Wire Line
+	8650 5250 8950 5250
+Wire Wire Line
+	8950 5250 8950 5200
+Wire Wire Line
+	8950 4900 8950 4800
+Connection ~ 8950 4800
+Wire Wire Line
+	8950 4800 9800 4800
+Wire Wire Line
+	8050 5250 8050 5500
+Connection ~ 8050 5500
+Wire Wire Line
+	8050 5500 9800 5500
+$Comp
+L Connector_Generic:Conn_01x02 CN?
+U 1 1 625E6ABC
+P 10950 5400
+AR Path="/625E6ABC" Ref="CN?"  Part="1"
+AR Path="/6188C66E/625E6ABC" Ref="CN?"  Part="1"
+AR Path="/6195E29D/625E6ABC" Ref="CN8"  Part="1"
+F 0 "CN8" V 10914 5212 50  0000 R CNN
+F 1 "CAN" V 10823 5212 50  0000 R CNN
+F 2 "telemetry-pcb:molex_sl_1x02_horizontal" H 10950 5400 50  0001 C CNN
+F 3 "~" H 10950 5400 50  0001 C CNN
+	1    10950 5400
+	1    0    0    -1
+$EndComp
+Wire Wire Line
+	10450 5500 10750 5500
+Connection ~ 10450 5500
+Wire Wire Line
+	10450 4900 10750 4900
+Wire Wire Line
+	10450 4900 10450 5500
+Wire Wire Line
+	9800 4800 10600 4800
+Wire Wire Line
+	10600 4800 10600 5400
+Wire Wire Line
+	10600 5400 10750 5400
+Connection ~ 10600 4800
+Wire Wire Line
+	10600 4800 10750 4800
 $EndSCHEMATC

Commit message: removes one power port, changes CAN switch to jumper
Parts:
- removed S2: CAN_TERM, Button_Switch_THT:SW_DIP_SPSTx01_Piano_10.8x4.1mm_W7.62mm_P2.54mm, symbol Switch:SW_DIP_x01
- added J3: CAN_TERM, Connector_PinHeader_2.54mm:PinHeader_1x02_P2.54mm_Horizontal, symbol Connector_Generic:Conn_01x02
Connections:
- wire segments 141 -> 142
Changed lines of the file:
@@
-$EndComp
-$Comp
-L Switch:SW_DIP_x01 S?
-U 1 1 62470711
-P 8350 5250
-AR Path="/62470711" Ref="S?"  Part="1"
-AR Path="/6188C66E/62470711" Ref="S?"  Part="1"
-AR Path="/6195E29D/62470711" Ref="S2"  Part="1"
-F 0 "S2" H 8350 5517 50  0000 C CNN
-F 1 "CAN_TERM" H 8350 5426 50  0000 C CNN
-F 2 "Button_Switch_THT:SW_DIP_SPSTx01_Piano_10.8x4.1mm_W7.62mm_P2.54mm" H 8350 5250 50  0001 C CNN
-F 3 "~" H 8350 5250 50  0001 C CNN
-	1    8350 5250
-	1    0    0    -1
 $EndComp
 $Comp
@@
 Wire Wire Line
 	9800 5500 10450 5500
-Wire Wire Line
-	8650 5250 8950 5250
 Wire Wire Line
 	8950 5250 8950 5200
@@
 Wire Wire Line
 	10600 4800 10750 4800
+$Comp
+L Connector_Generic:Conn_01x02 J3
+U 1 1 62267FF9
+P 8300 5050
+F 0 "J3" V 8264 4862 50  0000 R CNN
+F 1 "CAN_TERM" V 8173 4862 50  0000 R CNN
+F 2 "Connector_PinHeader_2.54mm:PinHeader_1x02_P2.54mm_Horizontal" H 8300 5050 50  0001 C CNN
+F 3 "~" H 8300 5050 50  0001 C CNN
+	1    8300 5050
+	0    -1   -1   0
+$EndComp
+Wire Wire Line
+	8400 5250 8950 5250
+Wire Wire Line
+	8050 5250 8300 5250
 $EndSCHEMATC

Commit message: Updates BOM
Parts:
- renumbered CN8 to CN2
Changed lines of the file:
@@
 AR Path="/625E6ABC" Ref="CN?"  Part="1"
 AR Path="/6188C66E/625E6ABC" Ref="CN?"  Part="1"
-AR Path="/6195E29D/625E6ABC" Ref="CN8"  Part="1"
-F 0 "CN8" V 10914 5212 50  0000 R CNN
+AR Path="/6195E29D/625E6ABC" Ref="CN2"  Part="1"
+F 0 "CN2" V 10914 5212 50  0000 R CNN
 F 1 "CAN" V 10823 5212 50  0000 R CNN
 F 2 "telemetry-pcb:molex_sl_1x02_horizontal" H 10950 5400 50  0001 C CNN

Commit message: deleted extraneous footprints
Parts:
- IC2, IC3: symbol telemetry-pcb-rescue:MAX31855K-telemetry-pcb-eagle-import-telemetry-pcb-rescue -> telemetry-pcb-rescue:MAX31855K-telemetry-pcb-eagle-import-telemetry-pcb-rescue-telemetry-pcb-rescue
- IC5: symbol telemetry-pcb-rescue:TCAN332DR-TCAN332DR-telemetry-pcb-rescue -> telemetry-pcb-rescue:TCAN332DR-TCAN332DR-telemetry-pcb-rescue-telemetry-pcb-rescue
- IC6: symbol telemetry-pcb-rescue:LSM6DSOTR-2021-11-02_20-37-28-telemetry-pcb-rescue-telemetry-pcb-rescue -> telemetry-pcb-rescue:LSM6DSOTR-2021-11-02_20-37-28-telemetry-pcb-rescue-telemetry-pcb-rescue-telemetry-pcb-rescue
Changed lines of the file:
@@
 $EndComp
 $Comp
-L telemetry-pcb-rescue:TCAN332DR-TCAN332DR-telemetry-pcb-rescue IC?
+L telemetry-pcb-rescue:TCAN332DR-TCAN332DR-telemetry-pcb-rescue-telemetry-pcb-rescue IC?
 U 1 1 6196EF6D
 P 7550 6650
@@
 $EndComp
 $Comp
-L telemetry-pcb-rescue:MAX31855K-telemetry-pcb-eagle-import-telemetry-pcb-rescue IC?
+L telemetry-pcb-rescue:MAX31855K-telemetry-pcb-eagle-import-telemetry-pcb-rescue-telemetry-pcb-rescue IC?
 U 1 1 6198C080
 P 2400 1450
@@
 	1000 1650 1900 1650
 $Comp
-L telemetry-pcb-rescue:LSM6DSOTR-2021-11-02_20-37-28-telemetry-pcb-rescue-telemetry-pcb-rescue IC?
+L telemetry-pcb-rescue:LSM6DSOTR-2021-11-02_20-37-28-telemetry-pcb-rescue-telemetry-pcb-rescue-telemetry-pcb-rescue IC?
 U 1 1 61D40F93
 P 8450 2750
@@
 	2200 3450 2200 4150
 $Comp
-L telemetry-pcb-rescue:MAX31855K-telemetry-pcb-eagle-import-telemetry-pcb-rescue IC?
+L telemetry-pcb-rescue:MAX31855K-telemetry-pcb-eagle-import-telemetry-pcb-rescue-telemetry-pcb-rescue IC?
 U 1 1 6198C07A
 P 3100 3450

Commit message: changes CAN ports to 3 pin, Thermocouple ports to 2 pin
Parts:
- CN2, CN7: footprint telemetry-pcb:molex_sl_1x02_horizontal -> telemetry-pcb:molex-sl-1x03-horizontal; symbol Connector_Generic:Conn_01x02 -> Connector_Generic:Conn_01x03
- CN5, CN6: footprint telemetry-pcb:molex-sl-1x03-horizontal -> telemetry-pcb:molex_sl_1x02_horizontal; symbol Connector_Generic:Conn_01x03 -> Connector_Generic:Conn_01x02
Connections:
- net GND: now also CN2.2 (Pin_2), CN7.2 (Pin_2)
- net at IC5.7 (CANH), J3.1 (Pin_1), T6.2 (Pin_2): now also CN2.3 (Pin_3), CN7.3 (Pin_3); no longer CN2.2 (Pin_2), CN7.2 (Pin_2)
- net at C8.1, IC3.2 (T-): now also CN6.2 (Pin_2); no longer CN6.3 (Pin_3)
- net at C7.1, IC2.2 (T-): now also CN5.2 (Pin_2); no longer CN5.3 (Pin_3)
- no-connect marks 12 -> 10
Other:
- moved on the sheet: T6
Changed lines of the file:
@@
 	1    0    0    -1
 $EndComp
-Wire Wire Line
-	650  1850 650  1950
-NoConn ~ 650  1750
-$Comp
-L Connector_Generic:Conn_01x03 CN?
+$Comp
+L Connector_Generic:Conn_01x02 CN?
 U 1 1 6198C0AA
 P 450 1750
@@
 F 0 "CN5" V 414 1562 50  0000 R CNN
 F 1 "THERMO1" V 323 1562 50  0000 R CNN
-F 2 "telemetry-pcb:molex-sl-1x03-horizontal" H 450 1750 50  0001 C CNN
+F 2 "telemetry-pcb:molex_sl_1x02_horizontal" H 450 1750 50  0001 C CNN
 F 3 "~" H 450 1750 50  0001 C CNN
 	1    450  1750
@@
 	1    0    0    -1
 $EndComp
-NoConn ~ 1300 3750
-Wire Wire Line
-	1300 3850 1300 3950
-$Comp
-L Connector_Generic:Conn_01x03 CN?
+$Comp
+L Connector_Generic:Conn_01x02 CN?
 U 1 1 6198C0A0
 P 1100 3750
@@
 F 0 "CN6" V 1064 3562 50  0000 R CNN
 F 1 "THERMO2" V 973 3562 50  0000 R CNN
-F 2 "telemetry-pcb:molex-sl-1x03-horizontal" H 1100 3750 50  0001 C CNN
+F 2 "telemetry-pcb:molex_sl_1x02_horizontal" H 1100 3750 50  0001 C CNN
 F 3 "~" H 1100 3750 50  0001 C CNN
 	1    1100 3750
@@
 L Connector:Conn_01x02_Female T?
 U 1 1 62470705
-P 10000 5100
+P 9800 5100
 AR Path="/62470705" Ref="T?"  Part="1"
 AR Path="/6188C66E/62470705" Ref="T?"  Part="1"
 AR Path="/6195E29D/62470705" Ref="T6"  Part="1"
-F 0 "T6" H 10028 5076 50  0000 L CNN
-F 1 "TEST_CAN" H 10028 4985 50  0000 L CNN
-F 2 "TestPoint:TestPoint_2Pads_Pitch2.54mm_Drill0.8mm" H 10000 5100 50  0001 C CNN
-F 3 "~" H 10000 5100 50  0001 C CNN
-	1    10000 5100
-	1    0    0    -1
-$EndComp
-$Comp
-L Connector_Generic:Conn_01x02 CN?
+F 0 "T6" H 9828 5076 50  0000 L CNN
+F 1 "TEST_CAN" H 9828 4985 50  0000 L CNN
+F 2 "TestPoint:TestPoint_2Pads_Pitch2.54mm_Drill0.8mm" H 9800 5100 50  0001 C CNN
+F 3 "~" H 9800 5100 50  0001 C CNN
+	1    9800 5100
+	1    0    0    -1
+$EndComp
+$Comp
+L Connector_Generic:Conn_01x03 CN?
 U 1 1 6247070B
-P 10950 4800
+P 10950 4900
 AR Path="/6247070B" Ref="CN?"  Part="1"
 AR Path="/6188C66E/6247070B" Ref="CN?"  Part="1"
 AR Path="/6195E29D/6247070B" Ref="CN7"  Part="1"
-F 0 "CN7" V 10914 4612 50  0000 R CNN
-F 1 "CAN" V 10823 4612 50  0000 R CNN
-F 2 "telemetry-pcb:molex_sl_1x02_horizontal" H 10950 4800 50  0001 C CNN
-F 3 "~" H 10950 4800 50  0001 C CNN
-	1    10950 4800
+F 0 "CN7" V 10914 4712 50  0000 R CNN
+F 1 "CAN" V 10823 4712 50  0000 R CNN
+F 2 "telemetry-pcb:molex-sl-1x03-horizontal" H 10950 4900 50  0001 C CNN
+F 3 "~" H 10950 4900 50  0001 C CNN
+	1    10950 4900
 	1    0    0    -1
 $EndComp
@@
 	6550 4800 6550 6550
 Wire Wire Line
-	9800 5200 9800 5500
-Wire Wire Line
-	9800 5100 9800 4800
-Connection ~ 9800 4800
-Connection ~ 9800 5500
+	9600 5200 9600 5500
+Wire Wire Line
+	9600 5100 9600 4800
 Wire Wire Line
 	6700 5500 8050 5500
 Wire Wire Line
 	6550 4800 8950 4800
-Wire Wire Line
-	9800 5500 10450 5500
 Wire Wire Line
 	8950 5250 8950 5200
@@
 Connection ~ 8950 4800
 Wire Wire Line
-	8950 4800 9800 4800
+	8950 4800 9600 4800
 Wire Wire Line
 	8050 5250 8050 5500
 Connection ~ 8050 5500
 Wire Wire Line
-	8050 5500 9800 5500
-$Comp
-L Connector_Generic:Conn_01x02 CN?
+	8050 5500 9600 5500
+$Comp
+L Connector_Generic:Conn_01x03 CN?
 U 1 1 625E6ABC
 P 10950 5400
@@
 F 0 "CN2" V 10914 5212 50  0000 R CNN
 F 1 "CAN" V 10823 5212 50  0000 R CNN
-F 2 "telemetry-pcb:molex_sl_1x02_horizontal" H 10950 5400 50  0001 C CNN
+F 2 "telemetry-pcb:molex-sl-1x03-horizontal" H 10950 5400 50  0001 C CNN
 F 3 "~" H 10950 5400 50  0001 C CNN
 	1    10950 5400
@@
 $EndComp
 Wire Wire Line
-	10450 5500 10750 5500
-Connection ~ 10450 5500
-Wire Wire Line
-	10450 4900 10750 4900
-Wire Wire Line
-	10450 4900 10450 5500
-Wire Wire Line
-	9800 4800 10600 4800
-Wire Wire Line
-	10600 4800 10600 5400
-Wire Wire Line
-	10600 5400 10750 5400
-Connection ~ 10600 4800
-Wire Wire Line
-	10600 4800 10750 4800
+	10500 4800 10500 5300
 $Comp
 L Connector_Generic:Conn_01x02 J3
@@
 Wire Wire Line
 	8050 5250 8300 5250
+Wire Wire Line
+	10350 5000 10350 5500
+$Comp
+L power:GND #PWR?
+U 1 1 62320513
+P 10650 6000
+AR Path="/62320513" Ref="#PWR?"  Part="1"
+AR Path="/6195E29D/62320513" Ref="#PWR0101"  Part="1"
+F 0 "#PWR0101" H 10650 5750 50  0001 C CNN
+F 1 "GND" H 10655 5827 50  0000 C CNN
+F 2 "" H 10650 6000 50  0001 C CNN
+F 3 "" H 10650 6000 50  0001 C CNN
+	1    10650 6000
+	1    0    0    -1
+$EndComp
+Wire Wire Line
+	10650 4900 10750 4900
+Wire Wire Line
+	10650 4900 10650 5400
+Wire Wire Line
+	10650 5400 10750 5400
+Connection ~ 10650 5400
+Wire Wire Line
+	10650 5400 10650 6000
+Wire Wire Line
+	1300 3750 1300 3950
+Wire Wire Line
+	650  1750 650  1950
+Connection ~ 9600 4800
+Connection ~ 9600 5500
+Wire Wire Line
+	9600 5500 10350 5500
+Wire Wire Line
+	9600 4800 10500 4800
+Connection ~ 10350 5500
+Wire Wire Line
+	10350 5500 10750 5500
+Connection ~ 10500 4800
+Wire Wire Line
+	10500 4800 10750 4800
+Wire Wire Line
+	10350 5000 10750 5000
+Wire Wire Line
+	10500 5300 10750 5300
 $EndSCHEMATC

Commit message: some more small changes from design review
Parts:
- CN5, CN6: footprint telemetry-pcb:molex_sl_1x02_horizontal -> telemetry-pcb:ScrewTermPlug1x02
Changed lines of the file:
@@
 F 0 "CN5" V 414 1562 50  0000 R CNN
 F 1 "THERMO1" V 323 1562 50  0000 R CNN
-F 2 "telemetry-pcb:molex_sl_1x02_horizontal" H 450 1750 50  0001 C CNN
+F 2 "telemetry-pcb:ScrewTermPlug1x02" H 450 1750 50  0001 C CNN
 F 3 "~" H 450 1750 50  0001 C CNN
 	1    450  1750
@@
 F 0 "CN6" V 1064 3562 50  0000 R CNN
 F 1 "THERMO2" V 973 3562 50  0000 R CNN
-F 2 "telemetry-pcb:molex_sl_1x02_horizontal" H 1100 3750 50  0001 C CNN
+F 2 "telemetry-pcb:ScrewTermPlug1x02" H 1100 3750 50  0001 C CNN
 F 3 "~" H 1100 3750 50  0001 C CNN
 	1    1100 3750
