File: serial.kicad_sch (KiCad schematic)
At the start: 13 parts

Commit message: fixed power flag in schematic causing error
Parts:
- C2, C3, C4, C5, C6: renamed from C?; value (none) -> 0.1uF; footprint (none) -> Capacitor_SMD:C_0805_2012Metric
- CN3: renamed from CN?; value (none) -> RS232; footprint (none) -> Connector_Dsub:DSUB-9_Female_Horizontal_P2.77x2.84mm_EdgePinOffset7.70mm_Housed_MountingHolesOffset9.12mm
- CN4: value (none) -> UART; footprint (none) -> telemetry-pcb:molex_sl_1x04_horizontal
- IC1: renamed from IC?; value (none) -> MAX3232CPWR; footprint (none) -> Package_SO:TSSOP-16_4.4x5mm_P0.65mm
- J1: value (none) -> TX_SEL; footprint (none) -> Connector_PinHeader_2.54mm:PinHeader_2x02_P2.54mm_Horizontal
- J2: value (none) -> RX_SEL; footprint (none) -> Connector_PinHeader_2.54mm:PinHeader_2x03_P2.54mm_Horizontal
- Q1: value (none) -> IF-D92; footprint (none) -> telemetry-pcb:IF-D92
- R7: value (none) -> 10K; footprint (none) -> Resistor_SMD:R_0805_2012Metric
- T5: renamed from T?; value (none) -> TEST_RS232; footprint (none) -> TestPoint:TestPoint_2Pads_Pitch2.54mm_Drill0.8mm

Commit message: 3.0 Preliminary Changes
Connections:
- net GND: now also CN3.5
- no-connect marks 11 -> 10

Commit message: Completed PCB routing
new footprints added to Footprints folder, added I2C peripherals page.
Parts:
- removed CN4: UART, telemetry-pcb:molex_sl_1x04_horizontal, symbol Connector_Generic:Conn_01x04
- added CN2: UART, Footprints:CONN_SD-43650-001_04_MOL, symbol telemetry_3.0_sch_library:436500400
Connections:
- net +3V3: now also CN2.4
- net GND: now also CN2.1
- net at J1.3 (Pin_3): now also CN2.3
- net at J2.3 (Pin_3): now also CN2.2
Other:
- moved on the sheet: C2, C3, C4, C5, C6, CN3, IC1, J1, J2, Q1, R7, T5
